File: power.kicad_sch (KiCad schematic)
At the start: 29 parts, among them J2 USB_C_Receptacle, Q1 Q_NMOS_GSD, Q2 Q_NMOS_GSD, Q3 DMG2301L, U3 MCP73831-2-OT, U4 MAX17048, U8 LD39150DT33

Commit message: PCB layout
Connections:
- net +BATT: no longer R7.1
- net at C7.1, R3.1, U2.2 (VDD): now also R7.1
- net D+ renamed D_P
- net D- renamed D_N

Commit message: Added LCSC PN for bms
Parts:
- U4: LCSC PN (none) -> C2682616
Changed lines of the file:
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@@
+			)
+		)
+		(property "LCSC PN" "C2682616"
+			(at 140.97 82.55 0)
+			(effects
+				(font
+					(size 1.27 1.27)
+				)
+				(hide yes)
 			)
 		)

Commit message: Made modifications from fabrication
Parts:
- BT1: MPN (none) -> C157932
- C10, C7: MPN (none) -> C14663
- C19, C20: MPN (none) -> C15849
- C8, C9, R7, R8: MPN (none) -> C19666
- D1, D4: value B340 -> SS34C; LCSC PN C64982 -> C13763; MPN (none) -> C13763
- D2: MPN (none) -> C965817
- D5: MPN (none) -> C48260
- F1: MPN (none) -> C135349
- J2: MPN (none) -> C2874568
- Q1, Q2: MPN (none) -> C260927
- Q3: MPN (none) -> C102619
- R1, R2: MPN (none) -> C122969
- R3: MPN (none) -> C107696
- R4, R5: MPN (none) -> C105576
- R6: MPN (none) -> C114669
- R9: MPN (none) -> C14675
- U2: MPN (none) -> C5881307
- U3: MPN (none) -> C424093
- U4: MPN (none) -> C2682616
- U8: MPN (none) -> C155559
